File: glass_udrive_pcb.brd (EAGLE design)
At the start: 14.5 x 19.9 mm, 23 parts

Commit message: minor routing and dimension and docu layer changes.
Routing:
- net GLASS_FLT: track 7.39 -> 5.63 mm
- net GLASS: track 12.3 -> 11.0 mm
- net GND: vias 5 -> 7
Other:
- board size 14.5 x 19.9 mm -> 15.4 x 19.9 mm
- board text added: "Head-plate mounting"
- board text added: "anchoring tab"
Changed lines of the file:
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@@
 <setting verticaltext="up"/>
 </settings>
-<grid distance="2" unitdist="mil" unit="mil" style="lines" multiple="1" display="yes" altdistance="0.01" altunitdist="mm" altunit="mm"/>
+<grid distance="0.2" unitdist="mm" unit="mm" style="lines" multiple="1" display="yes" altdistance="0.01" altunitdist="mm" altunit="mm"/>
 <layers>
 <layer number="1" name="Top" color="4" fill="1" visible="yes" active="yes"/>
@@
 <layer number="42" name="bRestrict" color="1" fill="10" visible="no" active="yes"/>
 <layer number="43" name="vRestrict" color="2" fill="10" visible="no" active="yes"/>
-<layer number="44" name="Drills" color="7" fill="1" visible="no" active="yes"/>
+<layer number="44" name="Drills" color="7" fill="1" visible="yes" active="yes"/>
 <layer number="45" name="Holes" color="7" fill="1" visible="yes" active="yes"/>
 <layer number="46" name="Milling" color="3" fill="1" visible="no" active="yes"/>
 <layer number="47" name="Measures" color="7" fill="1" visible="no" active="yes"/>
-<layer number="48" name="Document" color="7" fill="1" visible="no" active="yes"/>
+<layer number="48" name="Document" color="7" fill="1" visible="yes" active="yes"/>
 <layer number="49" name="Reference" color="7" fill="1" visible="no" active="yes"/>
 <layer number="50" name="dxf" color="7" fill="1" visible="no" active="no"/>
@@
 <board>
 <plain>
-<wire x1="-0.762" y1="-0.4064" x2="8.4328" y2="-0.4064" width="0.1" layer="20"/>
-<wire x1="8.5" y1="6.4636" x2="8.5" y2="19.508" width="0.1" layer="20"/>
+<wire x1="-1.5624" y1="-0.4064" x2="8.4328" y2="-0.4064" width="0.1" layer="20"/>
+<wire x1="8.49" y1="7.6436" x2="8.5" y2="19.508" width="0.1" layer="20"/>
 <wire x1="8.5" y1="19.508" x2="-0.762" y2="19.508" width="0.1" layer="20"/>
-<wire x1="-0.762" y1="19.508" x2="-0.762" y2="-0.4064" width="0.1" layer="20"/>
-<text x="7.2" y="8.1" size="0.5" layer="22" font="vector" rot="MR270">Nader Nikbakht
+<wire x1="-0.762" y1="19.508" x2="-0.762" y2="0.5524" width="0.1" layer="20"/>
+<wire x1="-0.762" y1="0.5524" x2="-1.5624" y2="0.5524" width="0.1" layer="20"/>
+<wire x1="-1.5624" y1="0.5524" x2="-1.5624" y2="-0.4064" width="0.1" layer="20"/>
+<text x="7" y="6.9" size="0.5" layer="22" font="vector" rot="MR270">Nader Nikbakht
 FeeLab, MIT 2018</text>
-<text x="4.9016" y="6.9618" size="0.5" layer="22" font="vector" rot="MR270">Glass uDrive
+<text x="5.6216" y="6.5818" size="0.5" layer="22" font="vector" rot="MR270">Glass uDrive
 Rev 1.0</text>
 <circle x="-12.827" y="-19.7104" radius="0.071840625" width="0.4064" layer="121"/>
@@
 </polygon>
 <wire x1="2.6816" y1="17.6058" x2="2.961" y2="17.3264" width="0.2032" layer="21"/>
-<wire x1="8.4328" y1="-0.4064" x2="8.4328" y2="3.2512" width="0.1016" layer="20"/>
-<wire x1="8.4328" y1="3.2512" x2="13.716" y2="3.2512" width="0.1016" layer="20"/>
-<wire x1="13.716" y1="3.2512" x2="13.706" y2="6.47" width="0.1016" layer="20"/>
-<wire x1="8.4944" y1="6.47" x2="13.706" y2="6.47" width="0.1016" layer="20"/>
-<dimension x1="8.4328" y1="0" x2="8.4328" y2="3.2512" x3="18.796" y3="1.6256" textsize="0.5" layer="20" width="0.01" visible="yes"/>
-<hole x="9.76" y="4.898" drill="1.5"/>
-<hole x="12.3" y="4.908" drill="1.5"/>
-<dimension x1="9.76" y1="4.4" x2="12.3" y2="4.4" x3="11.03" y3="6.988" textsize="0.5" layer="20" dtype="diameter" width="0.01" extwidth="0.01" visible="yes"/>
-<dimension x1="13.716" y1="5.588" x2="8.5044" y2="5.588" x3="11.1102" y3="8.124" textsize="0.5" layer="20" width="0.01" extwidth="0.01" visible="yes"/>
-<dimension x1="-0.762" y1="0" x2="13.716" y2="0" x3="6.477" y3="-1.778" textsize="0.5" layer="20" width="0.01" extwidth="0.01" visible="yes"/>
-<dimension x1="13.716" y1="3.2512" x2="13.706" y2="6.47" x3="14.5544" y3="4.86321875" textsize="0.5" layer="20" width="0.01" extwidth="0.01" visible="yes"/>
-<dimension x1="8.5" y1="19.508" x2="-0.762" y2="19.508" x3="3.869" y3="21.463" textsize="0.5" layer="20" width="0.01" extwidth="0.01" visible="yes"/>
-<dimension x1="-0.762" y1="-0.4064" x2="-0.762" y2="19.508" x3="-2.2352" y3="9.5508" textsize="0.508" layer="20" width="0.01" extwidth="0.01" visible="yes"/>
+<wire x1="8.4328" y1="-0.4064" x2="9.2456" y2="-0.4064" width="0.1016" layer="20"/>
+<wire x1="9.2456" y1="-0.4064" x2="9.2456" y2="0.6096" width="0.1016" layer="20"/>
+<wire x1="9.2456" y1="0.6096" x2="8.4328" y2="0.6096" width="0.1016" layer="20"/>
+<wire x1="8.4328" y1="0.6096" x2="8.43" y2="2.17" width="0.1016" layer="20"/>
+<wire x1="9.6" y1="3.25" x2="13.87" y2="3.2512" width="0.1016" layer="20"/>
+<wire x1="13.87" y1="3.2512" x2="13.87" y2="6.48" width="0.1016" layer="20"/>
+<dimension x1="-0.762" y1="0" x2="13.716" y2="0" x3="6.477" y3="-1.778" textsize="0.5" layer="51" width="0.01" extwidth="0.01" visible="yes"/>
+<dimension x1="8.5" y1="19.508" x2="-0.762" y2="19.508" x3="3.869" y3="21.463" textsize="0.5" layer="51" width="0.01" extwidth="0.01" visible="yes"/>
+<dimension x1="-0.762" y1="-0.4064" x2="-0.762" y2="19.508" x3="-2.2352" y3="9.5508" textsize="0.508" layer="51" width="0.01" extwidth="0.01" visible="yes"/>
+<dimension x1="-1.9544" y1="-0.4064" x2="-1.9544" y2="0.5896" x3="-1.3" y3="0.0916" textsize="0.508" layer="51" width="0.0254" extwidth="0.0254"/>
+<dimension x1="9.2456" y1="0.6096" x2="8.4328" y2="0.6096" x3="8.8392" y3="-2.6" textsize="0.508" layer="51" width="0.0254" extwidth="0.0254" visible="yes"/>
+<dimension x1="-0.7544" y1="0.6096" x2="-1.5672" y2="0.6096" x3="-1.1608" y3="-2.6" textsize="0.508" layer="51" width="0.0254" extwidth="0.0254" visible="yes"/>
+<dimension x1="13.97" y1="3.2512" x2="13.96" y2="6.47" x3="14.9001125" y3="4.86350625" textsize="0.508" layer="51" width="0.0254" extwidth="0.0254" visible="yes"/>
+<dimension x1="9.2456" y1="-0.4064" x2="9.2456" y2="0.6096" x3="10.2" y3="0.1016" textsize="0.508" layer="51" width="0.0254" extwidth="0.0254" visible="yes"/>
+<dimension x1="9.76" y1="4.89" x2="12.3" y2="4.89" x3="11.03" y3="7.19" textsize="0.3" layer="51" width="0.0254" extwidth="0.0254" visible="yes"/>
+<dimension x1="8.4944" y1="6.47" x2="13.86" y2="6.47" x3="11.1772" y3="8.1" textsize="0.508" layer="51" width="0.0254" extwidth="0.0254" visible="yes"/>
+<text x="9.4" y="-0.1" size="0.508" layer="51">anchoring tab</text>
+<text x="15.9" y="4.4" size="0.508" layer="51">Head-plate
+mounting</text>
+<wire x1="9.67" y1="6.49" x2="13.87" y2="6.48" width="0.1016" layer="20"/>
+<wire x1="9.61" y1="3.25" x2="8.43" y2="2.15" width="0.1016" layer="20" curve="90"/>
+<wire x1="8.49" y1="7.64" x2="9.67" y2="6.49" width="0.1016" layer="20" curve="90"/>
 </plain>
 <attributes>
@@
 <vertex x="-0.762" y="19.508"/>
 <vertex x="8.49" y="19.498"/>
+<vertex x="8.5344" y="6.4516"/>
+<vertex x="13.97" y="6.4516"/>
+<vertex x="13.97" y="3.302"/>
+<vertex x="8.4836" y="3.2512"/>
 <vertex x="8.43" y="-0.4064"/>
 <vertex x="-0.762" y="-0.4064"/>
@@
 <via x="1.7272" y="14.3256" extent="1-16" drill="0.254"/>
 <wire x1="1.7272" y1="14.3256" x2="1.6764" y2="14.3764" width="0.1016" layer="16"/>
+<via x="9.7536" y="4.8768" extent="1-16" drill="1.5"/>
+<via x="12.2936" y="4.8768" extent="1-16" drill="1.5"/>
 </signal>
 <signal name="CAP_COM">
@@
 <contactref element="BRIDGE" pad="1"/>
 <wire x1="0.729678125" y1="11.22309375" x2="0.7112" y2="11.22309375" width="0.1524" layer="1"/>
-<wire x1="0.7112" y1="11.22309375" x2="0.7112" y2="9.5504" width="0.1524" layer="1"/>
 <contactref element="CAPCOM" pad="1"/>
 <wire x1="0.729678125" y1="11.22309375" x2="0.53710625" y2="11.22309375" width="0.1524" layer="1"/>
 <wire x1="0.53710625" y1="11.22309375" x2="0.53710625" y2="12.9356" width="0.1524" layer="1"/>
-<wire x1="0.53710625" y1="12.9356" x2="0.2216" y2="12.9356" width="0.1524" layer="1"/>
-<wire x1="0.2216" y1="12.9356" x2="-0.1524" y2="13.3096" width="0.1524" layer="1"/>
-<wire x1="-0.1524" y1="13.3096" x2="-0.1524" y2="18.1638" width="0.1524" layer="1"/>
+<wire x1="0.53710625" y1="12.9356" x2="0.5772" y2="12.8848" width="0.1524" layer="1"/>
+<wire x1="0.5772" y1="12.8848" x2="-0.1524" y2="12.8832" width="0.1524" layer="1"/>
+<wire x1="-0.1524" y1="12.8832" x2="-0.1524" y2="18.1638" width="0.1524" layer="1"/>
 <wire x1="-0.1524" y1="18.1638" x2="0.3222" y2="18.6384" width="0.1524" layer="1"/>
 </signal>
@@
 <wire x1="0.316" y1="17.588" x2="0.2032" y2="17.4752" width="0.1016" layer="1"/>
 <wire x1="0.2032" y1="17.4752" x2="0.2032" y2="15.0368" width="0.1016" layer="1"/>
-<wire x1="0.2032" y1="15.0368" x2="0.2032" y2="13.26950625" width="0.1016" layer="1"/>
-<wire x1="0.8766" y1="15.0909" x2="0.2573" y2="15.0909" width="0.1016" layer="1"/>
-<wire x1="0.2573" y1="15.0909" x2="0.2032" y2="15.0368" width="0.1016" layer="1"/>
 <wire x1="0.8766" y1="15.0909" x2="1.5715" y2="15.0909" width="0.1016" layer="1"/>
 <wire x1="1.5715" y1="15.0909" x2="1.7272" y2="14.9352" width="0.1016" layer="1"/>
 <wire x1="1.7272" y1="14.9352" x2="2.6144" y2="14.9352" width="0.1016" layer="1"/>
 <wire x1="2.6144" y1="14.9352" x2="2.622" y2="14.9428" width="0.1016" layer="1"/>
+<wire x1="0.8766" y1="15.0909" x2="0.8225" y2="15.0368" width="0.1016" layer="1"/>
+<wire x1="0.8225" y1="15.0368" x2="0.2032" y2="15.0368" width="0.1016" layer="1"/>
 </signal>
 <signal name="REF_FLT">
@@
 <wire x1="6.178" y1="16.8732" x2="6.1722" y2="16.879" width="0.1524" layer="1"/>
 </signal>
+<signal name="N$1">
+</signal>
+<signal name="N$5">
+</signal>
 </signals>
