File: eaglefiles/glass_udrive_pcb.brd (EAGLE design)
At the start: 15.4 x 20 mm, 23 parts

Commit message: stuff and things
Parts:
- moved C4 1.68 mm to (0.01, 15.9), turned to 270 degrees
- moved CAPCOM 0.32 mm to (0.76, 12.9), turned to 180 degrees
- moved R2 0.16 mm to (0.77, 15.9), turned to 270 degrees
Routing:
- net GLASS_OUT: track 20.8 -> 2.30 mm
- net +15V: track 25.9 -> 8.05 mm
- net REF_FLT: track 14.2 -> 3.39 mm
- net GLASS_FLT: track 5.92 -> 3.03 mm
- net GLASS: track 10.9 -> 13.0 mm, vias 0 -> 1
- net GND: track 10.9 -> 12.8 mm
- net BRG_BAL: track 13.3 -> 12.5 mm
- net CAP_COM: track 14.9 -> 15.6 mm
